File: Hardware/SparkFun_MMA8452Q-Breakout.brd (EAGLE design)
At the start: 25.4 x 25.4 mm, 21 parts, among them J2 SMD, J3 PTH, J4 SMD, U2 MMA8452Q

Commit message: Added a GND via. Created 3mm spaced panel.
Parts:
- moved LOGO1 1.27 mm to (2.54, 3.81)
Routing:
- net GND: track 10.3 -> 12.8 mm, vias 5 -> 6
- net SCL: track 46.3 -> 46.9 mm
Other:
- board text added: "X01"
Changed lines of the file:
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@@
 <layer number="47" name="Measures" color="7" fill="1" visible="no" active="yes"/>
 <layer number="48" name="Document" color="7" fill="1" visible="no" active="yes"/>
-<layer number="49" name="Reference" color="7" fill="1" visible="yes" active="yes"/>
+<layer number="49" name="Reference" color="7" fill="1" visible="no" active="yes"/>
 <layer number="50" name="dxf" color="7" fill="1" visible="no" active="yes"/>
 <layer number="51" name="tDocu" color="6" fill="1" visible="yes" active="yes"/>
@@
 <wire x1="4.8768" y1="18.9738" x2="5.5118" y2="18.3388" width="0.1778" layer="22"/>
 <wire x1="5.5118" y1="18.9738" x2="4.8768" y2="18.3388" width="0.1778" layer="22"/>
+<text x="2.413" y="1.27" size="1.27" layer="16" font="vector" ratio="15" rot="MR0" align="center">X01</text>
 </plain>
 <attributes>
@@
 <attribute name="PROD_ID" value="RES-00824" x="12.7" y="8.89" size="1.778" layer="27" font="vector" ratio="15" display="off"/>
 </element>
-<element name="LOGO1" library="SparkFun-Aesthetics" package="OSHW-LOGO-MINI" value="OSHW-LOGOMINI" x="2.54" y="2.54" rot="MR0"/>
+<element name="LOGO1" library="SparkFun-Aesthetics" package="OSHW-LOGO-MINI" value="OSHW-LOGOMINI" x="2.54" y="3.81" rot="MR0"/>
 <element name="U$1" library="SparkX" package="SPARKX-MEDIUM" value="SPARKX-LOGO4" x="12.7" y="19.685" rot="MR0"/>
 </elements>
@@
 <contactref element="C1" pad="1"/>
 <contactref element="U2" pad="2"/>
-<wire x1="11.425" y1="13.2" x2="10.168" y2="13.2" width="0.1778" layer="1"/>
+<wire x1="11.275" y1="13.2" x2="10.168" y2="13.2" width="0.1778" layer="1"/>
 <wire x1="10.168" y1="13.2" x2="9.818" y2="13.55" width="0.1778" layer="1"/>
 <wire x1="8.89" y1="13.55" x2="9.818" y2="13.55" width="0.1778" layer="1"/>
@@
 <contactref element="J4" pad="2"/>
 <contactref element="R2" pad="2"/>
-<wire x1="12.7" y1="14.732" x2="12.7" y2="16.51" width="0.1778" layer="1"/>
 <wire x1="20.32" y1="12.2" x2="19.296" y2="12.2" width="0.1778" layer="1"/>
 <wire x1="19.296" y1="12.2" x2="19.05" y2="12.446" width="0.1778" layer="1"/>
@@
 <wire x1="16.51" y1="13.55" x2="15.787" y2="13.55" width="0.1778" layer="1"/>
 <wire x1="15.787" y1="13.55" x2="15.3035" y2="14.0335" width="0.1778" layer="1"/>
-<wire x1="15.3035" y1="14.0335" x2="14.605" y2="14.732" width="0.1778" layer="1"/>
-<wire x1="14.605" y1="14.732" x2="13.208" y2="14.732" width="0.1778" layer="1"/>
-<wire x1="13.208" y1="14.732" x2="12.7" y2="14.732" width="0.1778" layer="1"/>
-<wire x1="12.7" y1="14.732" x2="10.16" y2="14.732" width="0.1778" layer="1"/>
+<wire x1="15.3035" y1="14.0335" x2="14.351" y2="14.986" width="0.1778" layer="1"/>
 <wire x1="10.16" y1="14.732" x2="8.255" y2="14.732" width="0.1778" layer="1"/>
 <wire x1="8.255" y1="14.732" x2="6.723" y2="13.2" width="0.1778" layer="1"/>
 <wire x1="5.08" y1="13.2" x2="6.723" y2="13.2" width="0.1778" layer="1"/>
-<wire x1="11.425" y1="13.7" x2="10.43" y2="13.7" width="0.1778" layer="1"/>
+<wire x1="11.275" y1="13.7" x2="10.43" y2="13.7" width="0.1778" layer="1"/>
 <wire x1="10.43" y1="13.7" x2="10.16" y2="13.97" width="0.1778" layer="1"/>
 <wire x1="10.16" y1="13.97" x2="10.16" y2="14.732" width="0.1778" layer="1"/>
-<wire x1="13.2" y1="13.975" x2="13.2" y2="14.724" width="0.1778" layer="1"/>
-<wire x1="13.2" y1="14.724" x2="13.208" y2="14.732" width="0.1778" layer="1"/>
 <wire x1="13.55" y1="8.89" x2="13.55" y2="9.74" width="0.1778" layer="1"/>
 <wire x1="13.55" y1="9.74" x2="13.97" y2="10.16" width="0.1778" layer="1"/>
@@
 <wire x1="10.16" y1="5.08" x2="8.89" y2="3.81" width="0.1778" layer="1"/>
 <wire x1="8.89" y1="3.81" x2="8.89" y2="1.27" width="0.1778" layer="1"/>
+<wire x1="14.351" y1="14.986" x2="13.208" y2="14.986" width="0.1778" layer="1"/>
+<wire x1="13.208" y1="14.986" x2="12.7" y2="14.986" width="0.1778" layer="1"/>
+<wire x1="12.7" y1="14.986" x2="10.414" y2="14.986" width="0.1778" layer="1"/>
+<wire x1="10.414" y1="14.986" x2="10.16" y2="14.732" width="0.1778" layer="1"/>
+<wire x1="13.2" y1="14.125" x2="13.2" y2="14.978" width="0.1778" layer="1"/>
+<wire x1="13.2" y1="14.978" x2="13.208" y2="14.986" width="0.1778" layer="1"/>
+<wire x1="12.7" y1="16.51" x2="12.7" y2="14.986" width="0.1778" layer="1"/>
 </signal>
 <signal name="GND">
@@
 <via x="17.78" y="10.16" extent="1-16" drill="0.381"/>
 <via x="10.16" y="10.16" extent="1-16" drill="0.381"/>
-<wire x1="13.975" y1="12.2" x2="14.724" y2="12.2" width="0.1778" layer="1"/>
+<wire x1="14.125" y1="12.2" x2="14.724" y2="12.2" width="0.1778" layer="1"/>
 <wire x1="14.724" y1="12.2" x2="15.24" y2="11.684" width="0.1778" layer="1"/>
 <wire x1="15.24" y1="11.684" x2="15.24" y2="9.525" width="0.1778" layer="1"/>
@@
 <wire x1="17.145" y1="6.985" x2="17.78" y2="6.35" width="0.1778" layer="1"/>
 <via x="17.78" y="6.35" extent="1-16" drill="0.381"/>
-<wire x1="13.975" y1="13.2" x2="13.327" y2="13.2" width="0.1778" layer="1"/>
+<wire x1="14.125" y1="13.2" x2="13.327" y2="13.2" width="0.1778" layer="1"/>
 <wire x1="13.327" y1="13.2" x2="13.208" y2="13.081" width="0.1778" layer="1"/>
-<wire x1="13.975" y1="12.2" x2="13.327" y2="12.2" width="0.1778" layer="1"/>
+<wire x1="14.125" y1="12.2" x2="13.327" y2="12.2" width="0.1778" layer="1"/>
 <wire x1="13.327" y1="12.2" x2="13.208" y2="12.319" width="0.1778" layer="1"/>
 <wire x1="13.208" y1="12.319" x2="13.208" y2="13.081" width="0.1778" layer="1"/>
+<wire x1="11.275" y1="11.7" x2="10.684" y2="11.7" width="0.254" layer="1"/>
+<wire x1="10.684" y1="11.7" x2="10.541" y2="11.557" width="0.254" layer="1"/>
+<wire x1="10.541" y1="11.557" x2="10.541" y2="10.541" width="0.254" layer="1"/>
+<wire x1="10.541" y1="10.541" x2="10.16" y2="10.16" width="0.254" layer="1"/>
+<via x="20.32" y="17.78" extent="1-16" drill="0.381"/>
 </signal>
 <signal name="SCL">
@@
 <wire x1="16.51" y1="15.66" x2="17.614" y2="15.66" width="0.1778" layer="1"/>
 <wire x1="17.614" y1="15.66" x2="19.074" y2="14.2" width="0.1778" layer="1"/>
-<wire x1="11.425" y1="12.2" x2="10.168" y2="12.2" width="0.1778" layer="1"/>
+<wire x1="11.275" y1="12.2" x2="10.168" y2="12.2" width="0.1778" layer="1"/>
 <wire x1="10.168" y1="12.2" x2="9.779" y2="11.811" width="0.1778" layer="1"/>
 <wire x1="9.779" y1="11.811" x2="9.779" y2="11.049" width="0.1778" layer="1"/>
@@
 <wire x1="7.112" y1="10.414" x2="6.326" y2="11.2" width="0.1778" layer="1"/>
 <wire x1="5.08" y1="11.2" x2="6.326" y2="11.2" width="0.1778" layer="1"/>
-<wire x1="13.97" y1="1.27" x2="13.97" y2="2.54" width="0.1778" layer="16"/>
-<via x="10.16" y="7.62" extent="1-16" drill="0.381"/>
+<via x="8.89" y="7.62" extent="1-16" drill="0.381"/>
 <wire x1="20.32" y1="14.2" x2="22.63" y2="14.2" width="0.1778" layer="1"/>
 <wire x1="22.63" y1="14.2" x2="22.86" y2="13.97" width="0.1778" layer="1"/>
@@
 <wire x1="22.86" y1="13.97" x2="24.13" y2="12.7" width="0.1778" layer="16"/>
 <wire x1="24.13" y1="12.7" x2="24.13" y2="8.89" width="0.1778" layer="16"/>
+<wire x1="8.89" y1="10.414" x2="8.89" y2="7.62" width="0.1778" layer="1"/>
+<wire x1="20.32" y1="14.2" x2="19.074" y2="14.2" width="0.1778" layer="1"/>
+<wire x1="23.368" y1="8.128" x2="24.13" y2="8.89" width="0.1778" layer="16"/>
+<wire x1="13.97" y1="1.27" x2="13.97" y2="2.54" width="0.1778" layer="16"/>
 <wire x1="13.97" y1="2.54" x2="10.16" y2="6.35" width="0.1778" layer="16"/>
+<wire x1="23.368" y1="8.128" x2="10.668" y2="8.128" width="0.1778" layer="16"/>
+<wire x1="10.668" y1="8.128" x2="10.16" y2="7.62" width="0.1778" layer="16"/>
+<wire x1="10.16" y1="7.62" x2="8.89" y2="7.62" width="0.1778" layer="16"/>
 <wire x1="10.16" y1="6.35" x2="10.16" y2="7.62" width="0.1778" layer="16"/>
-<wire x1="8.89" y1="10.414" x2="8.89" y2="8.89" width="0.1778" layer="1"/>
-<wire x1="8.89" y1="8.89" x2="10.16" y2="7.62" width="0.1778" layer="1"/>
-<wire x1="20.32" y1="14.2" x2="19.074" y2="14.2" width="0.1778" layer="1"/>
-<wire x1="10.16" y1="7.62" x2="10.668" y2="8.128" width="0.1778" layer="16"/>
-<wire x1="10.668" y1="8.128" x2="23.368" y2="8.128" width="0.1778" layer="16"/>
-<wire x1="23.368" y1="8.128" x2="24.13" y2="8.89" width="0.1778" layer="16"/>
 </signal>
 <signal name="SDA">
@@
 <contactref element="U2" pad="6"/>
 <contactref element="J4" pad="3"/>
-<wire x1="12.2" y1="11.425" x2="12.2" y2="10.93" width="0.1778" layer="1"/>
+<wire x1="12.2" y1="11.275" x2="12.2" y2="10.93" width="0.1778" layer="1"/>
 <wire x1="20.32" y1="13.2" x2="22.36" y2="13.2" width="0.1778" layer="1"/>
 <wire x1="22.36" y1="13.2" x2="22.86" y2="12.7" width="0.1778" layer="1"/>
@@
 <contactref element="J1" pad="2"/>
 <contactref element="U2" pad="9"/>
-<wire x1="13.975" y1="11.7" x2="14.589" y2="11.7" width="0.1778" layer="1"/>
+<wire x1="14.125" y1="11.7" x2="14.589" y2="11.7" width="0.1778" layer="1"/>
 <wire x1="14.589" y1="11.7" x2="14.859" y2="11.43" width="0.1778" layer="1"/>
 <wire x1="14.859" y1="11.43" x2="14.859" y2="9.271" width="0.1778" layer="1"/>
@@
 <contactref element="J1" pad="1"/>
 <contactref element="U2" pad="11"/>
-<wire x1="13.975" y1="12.7" x2="14.986" y2="12.7" width="0.1778" layer="1"/>
+<wire x1="14.125" y1="12.7" x2="14.986" y2="12.7" width="0.1778" layer="1"/>
 <wire x1="15.621" y1="9.779" x2="19.05" y2="6.35" width="0.1778" layer="1"/>
 <wire x1="19.05" y1="6.35" x2="19.05" y2="1.27" width="0.1778" layer="1"/>
@@
 <contactref element="U2" pad="7"/>
 <contactref element="R2" pad="1"/>
-<wire x1="12.7" y1="11.425" x2="12.7" y2="10.287" width="0.1778" layer="1"/>
+<wire x1="12.7" y1="11.275" x2="12.7" y2="10.287" width="0.1778" layer="1"/>
 <wire x1="12.7" y1="10.287" x2="11.85" y2="9.437" width="0.1778" layer="1"/>
 <wire x1="11.85" y1="8.89" x2="11.85" y2="9.437" width="0.1778" layer="1"/>
